File: TESTESP1SH.brd (EAGLE design)
At the start: 86.4 x 53.3 mm, 29 parts, among them J1 Digital_0_7, J10 Power, J2 Analog, J3 Digital_8_13, J4 Analog, J5 Digital_0_7, J9 ESP01

Commit message: Changes for v2.0 release
Parts:
- removed J4: Analog, freetronics-master-v1:1X08
- removed J5: Digital_0_7, freetronics:1X08
- added JP1, JP2: (no value), freetronics-master-v1:1X02
- J2: device freetronics-master-v1:1X08 -> freetronics-master-v1.1:1X06
- moved R10 23.2 mm to (43.2, 21.6)
- moved R13 23.2 mm to (48.3, 21.6)
- moved R11 23.2 mm to (40.6, 21.6)
- moved R12 23.2 mm to (45.7, 21.6)
- moved R14 23.2 mm to (35.6, 21.6)
- moved R9 23.2 mm to (38.1, 21.6)
- moved R4 22.9 mm to (48.3, 7.62)
- moved R8 22.9 mm to (43.2, 7.62)
- moved R15 22.9 mm to (35.6, 7.62)
- moved R5 22.9 mm to (38.1, 7.62)
- moved R6 22.9 mm to (40.6, 7.62)
- moved R7 22.9 mm to (45.7, 7.62)
- moved R1 19.1 mm to (48.3, 35.8)
- moved R2 19.1 mm to (48.3, 46.0)
- moved R3 10.2 mm to (48.3, 40.9)
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Connections:
- removed net A10: J4.3, R6.1
- removed net A11: J4.4, R8.2
- removed net A12: J4.5, R7.2
- removed net A13: J4.6, R4.1
- removed net A14: J4.7
- removed net A15: J4.8
- removed net A6: J2.7
- removed net A7: J2.8
- removed net A8: J4.1, R15.2
- removed net A9: J4.2, R5.1
- removed net D14: J5.8
- removed net D15: J5.7
- removed net D16: J5.6
- removed net D17: J5.5
- removed net D18: J5.4
- removed net D19: J5.3, R3.1
- removed net D20: J5.2, R2.1
- removed net D21: J5.1, R1.1
- net A0: now also R15.2
- net A1: now also R5.1
- net A2: now also R6.1
- net A3: now also R8.2
- net A4: now also R7.2
- net A5: now also R4.1
- net D4: now also R2.1
- net D5: now also R3.1
- net D6: now also R1.1
Routing:
- net D6: track 0.00 -> 28.9 mm
- net D21: track 27.8 -> 0.00 mm
- net 5V: track 69.5 -> 42.8 mm
- net D5: track 0.00 -> 21.2 mm
- net N$3: track 2.92 -> 22.0 mm
- net N$2: track 2.92 -> 22.0 mm
- net D19: track 15.6 -> 0.00 mm
- net D4: track 0.00 -> 13.6 mm
- net N$5: track 31.3 -> 43.0 mm
- net N$8: track 22.6 -> 33.3 mm
- net N$9: track 38.4 -> 48.5 mm
- net N$7: track 28.7 -> 38.9 mm
- net N$6: track 30.2 -> 40.4 mm
- net N$4: track 32.8 -> 42.9 mm
- net N$1: track 3.56 -> 9.91 mm
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Other:
- board text added: "v2.0"
- board text removed: "A10"
- board text removed: "A11"
- board text removed: "A12"
- board text removed: "A13"
- board text removed: "A14"
- board text removed: "A15"
- board text removed: "A6"
- board text removed: "A7"
- board text removed: "A8"
- board text removed: "A9"
- board text removed: "D14"
- board text removed: "D15"
- board text removed: "D16"
- board text removed: "D17"
- board text removed: "D18"
- board text removed: "D19"
- board text removed: "D20"
- board text removed: "D21"
- board text removed: "v1.0"
