File: TESTESP1SH.sch (EAGLE design)
At the start: 29 parts, among them J1 Digital_0_7, J10 Power, J2 Analog, J3 Digital_8_13, J4 Analog, J5 Digital_0_7, J9 ESP01

Commit message: Changes for v2.0 release
Parts:
- removed J4: Analog, freetronics-master-v1:M08
- removed J5: Digital_0_7, freetronics:M08
- added JP1, JP2: (no value), freetronics-master-v1:M02PTH
- J2: device freetronics-master-v1:M08 -> freetronics-master-v1.1:M06SIP
Connections:
- removed net A10: J4.3, R6.1
- removed net A11: J4.4, R8.2
- removed net A12: J4.5, R7.2
- removed net A13: J4.6, R4.1
- removed net A14: J4.7
- removed net A15: J4.8
- removed net A6: J2.7
- removed net A7: J2.8
- removed net A8: J4.1, R15.2
- removed net A9: J4.2, R5.1
- removed net D14: J5.8
- removed net D15: J5.7
- removed net D16: J5.6
- removed net D17: J5.5
- removed net D18: J5.4
- removed net D19: J5.3, R3.1
- removed net D20: J5.2, R2.1
- removed net D21: J5.1, R1.1
- net A0: now also R15.2
- net A1: now also R5.1
- net A2: now also R6.1
- net A3: now also R8.2
- net A4: now also R7.2
- net A5: now also R4.1
- net D4: now also R2.1
- net D5: now also R3.1
- net D6: now also R1.1
Other:
- note added: "V2.0 (2017-03-22)"
- note added: "const int reflash_readback_pin = A0; // 20k pullup (and 1k in series) GPIO0 const int rst_readback_pin = A1; // 20k pullup (and 1k in series) const int vcc_readback_pin = A2; // 20k pulldown (and 1k in series) const int gnd_readback_pin = A3; // 20k pullup (and 1k in series) const int rx_readback_pin = A4; // 82.5k pulldown (and 1k in series) const int tx_readback_pin = A5; // 82.5k pulldown (and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"
- note removed: "V1.0 (2017-03-22)"
- note removed: "const int reflash_readback_pin = A8; // 20k pullup (and 1k in series) GPIO0 const int rst_readback_pin = A9; // 20k pullup (and 1k in series) const int vcc_readback_pin = A10; // 20k pulldown (and 1k in series) const int gnd_readback_pin = A11; // 20k pullup (and 1k in series) const int rx_readback_pin = A12; // 82.5k pulldown (and 1k in series) const int tx_readback_pin = A13; // 82.5k pulldown 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"
